File: KiCad/FaderWing.kicad_pcb (KiCad board)
At the start: 2 copper layers, 103 x 222.5 mm, 185 parts, among them J1 USB_C_Receptacle_USB2.0, SW1 Encoder_Switch, SW10 SW_Push, SW11 Encoder_Switch, SW12 SW_Push, SW13 SW_Push, SW14 SW_Push, SW15 SW_Push, SW16 Encoder_Switch, SW17 SW_Push, SW18 SW_Push, SW19 SW_Push, SW2 SW_Push, SW20 SW_Push, SW21 Encoder_Switch, SW22 SW_Push, SW23 SW_Push, SW24 SW_Push, SW25 SW_Push, SW3 SW_Push, SW4 SW_Push, SW5 SW_Push, SW6 Encoder_Switch, SW7 SW_Push, SW8 SW_Push, SW9 SW_Push, U1 USBLC6-2SC6, U2 STM32G473RCTx, U3 AP2161WG-7, U4 MIC5504-3.3YM5, U5 TXS0102DCU

Commit message: PCB Revision 0.5
Parts:
- C10, C11, C12, C13, C14, C15, C16, C17, C18, C19, C20, C21, C22, C23, C24, C25, C26, C27, C58, C59, C60, C61, C62, C63, C64, C65, C66, C67, C68, C69, C70, C71, C72, C9, D1, D10, D11, D12, D13, D14, D15, D17, D18, D19, D2, D20, D21, D22, D23, D24, D25, D26, D3, D4, D5, D6, D7, D8, D9, J1, R1, R2, R3, R4, TP12, TP13, TP14, TP15, TP16, TP17, TP18, TP19, TP20, TP21, TP26, TP27, TP28, TP29, TP30, U1, U2, U3, U4, U5: moved to F.Cu
- moved C53 400.8 mm to (124.0, 241.8), turned to -90 degrees
- moved C33 400.6 mm to (124.0, 79.8), turned to -90 degrees
- moved C43 399.0 mm to (122.5, 195.8), turned to -90 degrees
- moved D52 392.1 mm to (115.0, 243.5), turned to 0 degrees
- moved D32 391.9 mm to (115.0, 81.5), turned to 0 degrees
- moved D42 391.8 mm to (115.0, 197.5), turned to 0 degrees
- moved TP21 364.8 mm to (121.9, 249.0), turned to 180 degrees
- moved C54 362.0 mm to (104.0, 241.8), turned to -90 degrees
- moved C34 361.8 mm to (104.0, 79.8), turned to -90 degrees
- moved C44 360.2 mm to (102.5, 195.8), turned to -90 degrees
- moved D53 353.4 mm to (95.0, 243.5), turned to 0 degrees
- moved D33 353.2 mm to (95.0, 81.5), turned to 0 degrees
- moved D43 353.1 mm to (95.0, 197.5), turned to 0 degrees
- moved TP15 348.8 mm to (101.9, 249.0), turned to 180 degrees
- moved TP16 346.7 mm to (125.5, 233.2), turned to -90 degrees
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Routing:
- net GND: track 57.3 -> 1134.2 mm, vias 126 -> 77
- net Encoder5B: track 241.1 -> 64.9 mm
- net Encoder5A: track 235.0 -> 62.2 mm
- net Encoder3B: track 208.3 -> 37.2 mm
- net Encoder4B: track 225.1 -> 56.6 mm
- net Encoder3A: track 202.1 -> 36.8 mm
- net Fader1: track 55.9 -> 218.8 mm, vias 0 -> 2
- net Encoder4A: track 218.7 -> 55.8 mm
- net Fader2: track 39.0 -> 200.7 mm, vias 0 -> 2
- net Fader3: track 53.7 -> 182.9 mm, vias 0 -> 2
- net Row1: track 215.5 -> 341.7 mm, vias 1 -> 2
- net Row2: track 187.4 -> 313.2 mm, vias 1 -> 2
- net Row5: track 277.5 -> 155.9 mm, vias 1 -> 2
- net Encoder1B: track 165.8 -> 67.3 mm, vias 1 -> 2
- net Encoder2B: track 181.8 -> 83.5 mm, vias 1 -> 2
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Other:
- board size 103 x 222.5 mm -> 104 x 236 mm
- board text added: "Revision: ${REV} DIY MA3 Fader Wing - Open Source Hardware https://github.com/leocb/MA3-Fader-Wing"
- board text removed: "DIY MA3 Fader Wing - Open Source Hardware https://github.com/leocb/MA3-Fader-Wing Revision: ${REV}"

Commit message: Update to revision 0.7
Parts:
- added A-F1: TestPoint_Small, TestPoint:TestPoint_THTPad_D2.0mm_Drill1.0mm, B.Cu at (63.7, 112.0)
- added A-F2: TestPoint_Small, TestPoint:TestPoint_THTPad_D2.0mm_Drill1.0mm, B.Cu at (66.3, 112.0)
- added A-F3: TestPoint_Small, TestPoint:TestPoint_THTPad_D2.0mm_Drill1.0mm, B.Cu at (82.5, 112.0)
- added A-F4: TestPoint_Small, TestPoint:TestPoint_THTPad_D2.0mm_Drill1.0mm, B.Cu at (85.0, 112.0)
- added A-F5: TestPoint_Small, TestPoint:TestPoint_THTPad_D2.0mm_Drill1.0mm, B.Cu at (87.5, 112.0)
- added A-VDDA: TestPoint_Small, TestPoint:TestPoint_THTPad_D2.0mm_Drill1.0mm, B.Cu at (46.2, 112.1)
- added A-VSSA: TestPoint_Small, TestPoint:TestPoint_THTPad_D2.0mm_Drill1.0mm, B.Cu at (43.7, 112.1)
- added B-F1: TestPoint_Small, TestPoint:TestPoint_THTPad_D2.0mm_Drill1.0mm, B.Cu at (63.7, 122.5)
- added B-F2: TestPoint_Small, TestPoint:TestPoint_THTPad_D2.0mm_Drill1.0mm, B.Cu at (66.3, 122.5)
- added B-F3: TestPoint_Small, TestPoint:TestPoint_THTPad_D2.0mm_Drill1.0mm, B.Cu at (82.5, 122.5)
- added B-F4: TestPoint_Small, TestPoint:TestPoint_THTPad_D2.0mm_Drill1.0mm, B.Cu at (85.0, 122.5)
- added B-F5: TestPoint_Small, TestPoint:TestPoint_THTPad_D2.0mm_Drill1.0mm, B.Cu at (87.5, 122.5)
- added B-VDDA: TestPoint_Small, TestPoint:TestPoint_THTPad_D2.0mm_Drill1.0mm, B.Cu at (46.2, 122.6)
- added B-VSSA: TestPoint_Small, TestPoint:TestPoint_THTPad_D2.0mm_Drill1.0mm, B.Cu at (43.7, 122.6)
- added PA10: TestPoint_Small, TestPoint:TestPoint_Pad_D1.0mm, F.Cu at (63.0, 21.0)
- added PA3: TestPoint_Small, TestPoint:TestPoint_Pad_D1.0mm, F.Cu at (79.1, 25.0)
- added PB0: TestPoint_Small, TestPoint:TestPoint_Pad_D1.0mm, F.Cu at (80.2, 18.5)
- added PB1: TestPoint_Small, TestPoint:TestPoint_Pad_D1.0mm, F.Cu at (78.3, 17.4)
- added PB2: TestPoint_Small, TestPoint:TestPoint_Pad_D1.0mm, F.Cu at (78.2, 19.7)
- added PB9: TestPoint_Small, TestPoint:TestPoint_Pad_D1.0mm, F.Cu at (65.5, 36.0)
- added PC10: TestPoint_Small, TestPoint:TestPoint_Pad_D1.0mm, F.Cu at (57.8, 32.9)
- added PC11: TestPoint_Small, TestPoint:TestPoint_Pad_D1.0mm, F.Cu at (59.7, 33.5)
- added PC12: TestPoint_Small, TestPoint:TestPoint_Pad_D1.0mm, F.Cu at (61.7, 33.8)
- added PC13: TestPoint_Small, TestPoint:TestPoint_Pad_D1.0mm, F.Cu at (69.8, 37.6)
- added PC14: TestPoint_Small, TestPoint:TestPoint_Pad_D1.0mm, F.Cu at (71.8, 38.1)
- added PC15: TestPoint_Small, TestPoint:TestPoint_Pad_D1.0mm, F.Cu at (73.8, 37.6)
- added PC5: TestPoint_Small, TestPoint:TestPoint_Pad_D1.0mm, F.Cu at (80.5, 20.5)
- added PD2: TestPoint_Small, TestPoint:TestPoint_Pad_D1.0mm, F.Cu at (63.7, 33.8)
- added PF0: TestPoint_Small, TestPoint:TestPoint_Pad_D1.0mm, F.Cu at (75.5, 36.5)
- added PF1: TestPoint_Small, TestPoint:TestPoint_Pad_D1.0mm, F.Cu at (75.0, 34.5)
- added mouse-bite-1mm-slot: VAL**, Custom:mouse-bite-1mm-slot, F.Cu at (95.0, 116.5)
- added mouse-bite-1mm-slot: VAL**, Custom:mouse-bite-1mm-slot, F.Cu at (122.5, 178.0)
- added mouse-bite-1mm-slot: VAL**, Custom:mouse-bite-1mm-slot, F.Cu at (27.5, 178.0)
- added mouse-bite-1mm-slot: VAL**, Custom:mouse-bite-1mm-slot, F.Cu at (122.5, 138.0)
- added mouse-bite-1mm-slot: VAL**, Custom:mouse-bite-1mm-slot, F.Cu at (27.5, 138.0)
- added mouse-bite-1mm-slot: VAL**, Custom:mouse-bite-1mm-slot, F.Cu at (55.0, 116.5)
- moved C27 102.6 mm to (81.8, 17.9), turned to 90 degrees
- moved C23 99.4 mm to (82.0, 24.5), turned to 0 degrees
- moved C26 97.0 mm to (83.2, 17.9), turned to 90 degrees
- moved C24 94.4 mm to (83.5, 22.8), turned to 0 degrees
- moved C25 92.4 mm to (83.5, 21.5), turned to 0 degrees
- moved TP12 6.94 mm to (35.0, 249.0)
- moved TP13 6.94 mm to (55.0, 249.0)
- moved TP14 6.94 mm to (75.0, 249.0)
- moved TP15 6.94 mm to (95.0, 249.0)
- moved TP21 6.94 mm to (115.0, 249.0)
- moved C43 4.47 mm to (120.0, 199.5), turned to 90 degrees
- moved C44 4.47 mm to (100.0, 199.5), turned to 90 degrees
- moved C45 4.47 mm to (80.0, 199.5), turned to 90 degrees
- moved C46 4.47 mm to (60.0, 199.5), turned to 90 degrees
- moved C47 4.47 mm to (40.0, 199.5), turned to 90 degrees
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Connections:
- U2 pad 17: unconnected-(U2-PA3-Pad17) -> Net-(U2-PA3)
- U2 pad 2: unconnected-(U2-PC13-Pad2) -> Net-(U2-PC13)
- U2 pad 23: unconnected-(U2-PC5-Pad23) -> Net-(U2-PC5)
- U2 pad 24: unconnected-(U2-PB0-Pad24) -> Net-(U2-PB0)
- U2 pad 25: unconnected-(U2-PB1-Pad25) -> Net-(U2-PB1)
- U2 pad 26: unconnected-(U2-PB2-Pad26) -> Net-(U2-PB2)
- U2 pad 3: unconnected-(U2-PC14-Pad3) -> Net-(U2-PC14)
- U2 pad 4: unconnected-(U2-PC15-Pad4) -> Net-(U2-PC15)
- U2 pad 44: unconnected-(U2-PA10-Pad44) -> Net-(U2-PA10)
- U2 pad 5: unconnected-(U2-PF0-Pad5) -> Net-(U2-PF0)
- U2 pad 52: unconnected-(U2-PC10-Pad52) -> Net-(U2-PC10)
- U2 pad 53: unconnected-(U2-PC11-Pad53) -> Net-(U2-PC11)
- U2 pad 54: unconnected-(U2-PC12-Pad54) -> Net-(U2-PC12)
- U2 pad 55: unconnected-(U2-PD2-Pad55) -> Net-(U2-PD2)
- U2 pad 6: unconnected-(U2-PF1-Pad6) -> Net-(U2-PF1)
- U2 pad 62: unconnected-(U2-PB9-Pad62) -> Net-(U2-PB9)
Routing:
- net GND: track 1134.2 -> 710.2 mm, vias 77 -> 86
- net Col5: track 294.1 -> 446.3 mm
- net Col4: track 278.5 -> 391.5 mm
- net Col3: track 283.1 -> 351.1 mm
- net Fader5: track 148.3 -> 206.4 mm, vias 2 -> 1
- net VREF: track 335.1 -> 384.8 mm
- net Col2: track 276.8 -> 312.3 mm
- net Fader4: track 165.3 -> 189.6 mm, vias 2 -> 1
- net Net-(U2-PB1): track 0.00 -> 9.02 mm
- net Net-(U2-PC10): track 0.00 -> 8.71 mm
- net Net-(U2-PB0): track 0.00 -> 7.96 mm
- net Fader3: track 182.9 -> 175.5 mm, vias 2 -> 1
- net Net-(U2-PC11): track 0.00 -> 7.26 mm
- net Net-(U2-PC5): track 0.00 -> 6.54 mm
- net Net-(U2-PC14): track 0.00 -> 6.52 mm
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Other:
- board size 104 x 236 mm -> 108 x 240 mm
- board text added: "DIY MA3 Fader Wing Revision: ${REV} github.com/leocb/MA3-Fader-Wing"
- board text added: "JLCJLCJLCJLCJLC"
- board text removed: "Bolo de cenoura: Ingredientes: 3 cenouras médias raspadas e picadas 3 ovos 1 xícara de açúcar 1 e 1/2 xícaras de farinha de trigo 1/2 xícara de óleo vegetal 1 colher de chá de fermento em pó 1 colher de chá de bicarbonato de sódio 1 colher de chá de canela em pó (opcional) Instruções: - Pré-aqueça o forno a 180 graus Celsius. - Em uma tigela grande, bata os ovos com o açúcar até obter uma mistura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"
- board text removed: "Revision: ${REV} DIY MA3 Fader Wing - Open Source Hardware https://github.com/leocb/MA3-Fader-Wing"
