File: KiCad/FaderWing.kicad_pcb (KiCad board)
At the start: 2 copper layers, 108 x 240 mm, 242 parts, among them J1 USB_C_Receptacle_USB2.0, SW1 Encoder_Switch, SW10 SW_Push, SW11 Encoder_Switch, SW12 SW_Push, SW13 SW_Push, SW14 SW_Push, SW15 SW_Push, SW16 Encoder_Switch, SW17 SW_Push, SW18 SW_Push, SW19 SW_Push, SW2 SW_Push, SW20 SW_Push, SW21 Encoder_Switch, SW22 SW_Push, SW23 SW_Push, SW24 SW_Push, SW25 SW_Push, SW3 SW_Push, SW4 SW_Push, SW5 SW_Push, SW6 Encoder_Switch, SW7 SW_Push, SW8 SW_Push, SW9 SW_Push, U1 USBLC6-2SC6, U2 STM32G473RCTx, U3 AP2161WG-7, U4 MIC5504-3.3YM5, U5 TXS0102DCU

Commit message: Improve components routing
Parts:
- removed 3.3V, 5V: LED_Small, LED_SMD:LED_1206_3216Metric
- removed 3vNz, 5vNz: TestPoint_Small, TestPoint:TestPoint_Pad_D1.0mm
- added 3vNz1: TestPoint_Small, TestPoint:TestPoint_Pad_D1.0mm, F.Cu at (53.2, 38.5)
- added 5vNz1: TestPoint_Small, TestPoint:TestPoint_Pad_D1.0mm, F.Cu at (43.9, 38.5)
- added LED-3V1: LED_Small, LED_SMD:LED_1206_3216Metric, F.Cu at (53.0, 29.0)
- added LED-5V1: LED_Small, LED_SMD:LED_1206_3216Metric, F.Cu at (53.0, 23.0)
- moved R9 7.77 mm to (26.0, 244.8), turned to -90 degrees
- moved R7 5.24 mm to (56.2, 28.8), turned to 0 degrees
- moved C11 2.02 mm to (61.0, 27.0)
- moved C9 0.55 mm to (70.0, 35.1), turned to -90 degrees
- moved C13 0.06 mm to (50.8, 32.0)
- renumbered PB9 to PB10
Routing:
- net VREF: track 272.7 -> 257.8 mm, vias 5 -> 2
- net GND: track 484.8 -> 490.0 mm, vias 130 -> 145
- net Net-(LED-3V1-K): track 6.58 -> 2.75 mm
- net BOOT 0: track 42.7 -> 45.7 mm
- net JTDI: track 40.8 -> 43.3 mm
- net Net-(D56-DOUT): track 6.60 -> 8.77 mm
- net LED NRZs: track 10.1 -> 8.20 mm
- net Net-(U2-PB2): track 14.0 -> 12.5 mm
- net Col2: track 311.2 -> 309.8 mm
- net LED NRZ: track 32.3 -> 31.0 mm
- net Encoder1A: track 59.7 -> 58.5 mm
- net Encoder4A: track 61.7 -> 62.9 mm
- net Col3: track 347.9 -> 346.9 mm
- net JTDO: track 56.9 -> 56.2 mm
- net SWCLK: track 38.4 -> 39.0 mm
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Other:
- board text added: "1"
- board text added: "2"
- board text added: "3"
- board text added: "3vNz"
- board text added: "4"
- board text added: "5"
- board text added: "5V"
- board text added: "5vNz"
- board text added: "FADER"
- board text added: "|1|"
- board text added: "|2|"
- board text added: "|3|"
- board text added: "|4|"
- board text added: "|5|"
- board text removed: "FADERS"
